Commit message: ros_control: added right leg(need updating), head and torso

File: ar600_description/urdf/base/base.transmission.xacro (robot description, xacro)
@@ -3,13 +3,12 @@
   <xacro:macro name="ar600_base_torso_transmission">
     <transmission name="torso_rotation_trans">
-      <!-- <actuator name="torso_rotation_motor" /> -->
-      <joint name="torso_rotation_joint" />
-      <type>
-      	transmission_interface/SimpleTransmission
-      </type>
+      <type>transmission_interface/SimpleTransmission</type>
+      <joint name="torso_rotation_joint">
+        <hardwareInterface>EffortJointInterface</hardwareInterface>
+      </joint>
       <actuator name="torso_rotation_joint_actuator">
+        <hardwareInterface>EffortJointInterface</hardwareInterface>
         <mechanicalReduction>1</mechanicalReduction>
         <motorTorqueConstant>10</motorTorqueConstant>
-        <hardwareInterface>EffortJointInterface</hardwareInterface>
       </actuator>
       <!-- <mechanicalReduction>${-1 * 624/35 * 80/18}</mechanicalReduction> -->

File: ar600_description/urdf/base/base.urdf.xacro (robot description, xacro)
@@ -2,5 +2,5 @@
 <robot xmlns:xacro="http://ros.org/wiki/xacro">
   	<xacro:include filename="$(find ar600_description)/urdf/base/base.gazebo.xacro" />
-  	<!--<xacro:include filename="$(find ar600_description)/urdf/base/base.transmission.xacro" />-->
+  	<xacro:include filename="$(find ar600_description)/urdf/base/base.transmission.xacro" />
 	<xacro:macro name="ar600_body_macro" params="name">
 		<link name="${name}_link">
@@ -54,5 +54,5 @@
 		<xacro:ar600_base_gazebo name="${name}"/>
 		<xacro:ar600_torso_gazebo name="${name}"/>
-    	<!--<xacro:ar600_base_torso_transmission/>-->
+    	<xacro:ar600_base_torso_transmission/>
 	</xacro:macro>
 </robot>

File: ar600_description/urdf/head/head.transmission.xacro (robot description, xacro)
@@ -3,39 +3,36 @@
   <xacro:macro name="ar600_head_transmission">
     <transmission name="head_mount_transmission">
-      <!-- <actuator name="torso_rotation_motor" /> -->
-      <joint name="torso_head_mount" />
-      <type>
-      	transmission_interface/SimpleTransmission
-      </type>
+      <type>transmission_interface/SimpleTransmission</type>
+      <joint name="torso_head_mount">
+        <hardwareInterface>EffortJointInterface</hardwareInterface>
+      </joint>
       <actuator name="head_mount_joint_actuator">
+        <hardwareInterface>EffortJointInterface</hardwareInterface>
         <mechanicalReduction>1</mechanicalReduction>
         <motorTorqueConstant>10</motorTorqueConstant>
-        <hardwareInterface>EffortJointInterface</hardwareInterface>
       </actuator>
       <!-- <mechanicalReduction>${-1 * 624/35 * 80/18}</mechanicalReduction> -->
     </transmission>
 	<transmission name="mount_head_tilt_mount_transmission">
-      <!-- <actuator name="torso_rotation_motor" /> -->
-      <joint name="mount_head_tilt_mount" />
-      <type>
-      	transmission_interface/SimpleTransmission
-      </type>
+      <type>transmission_interface/SimpleTransmission</type>
+      <joint name="mount_head_tilt_mount">
+        <hardwareInterface>EffortJointInterface</hardwareInterface>
+      </joint>
       <actuator name="mount_head_tilt_mount_joint_actuator">
+        <hardwareInterface>EffortJointInterface</hardwareInterface>
         <mechanicalReduction>1</mechanicalReduction>
         <motorTorqueConstant>10</motorTorqueConstant>
-        <hardwareInterface>EffortJointInterface</hardwareInterface>
       </actuator>
       <!-- <mechanicalReduction>${-1 * 624/35 * 80/18}</mechanicalReduction> -->
     </transmission>
 	<transmission name="head_mount_head_transmission">
-      <!-- <actuator name="torso_rotation_motor" /> -->
-      <joint name="head_mount_head" />
-      <type>
-      	transmission_interface/SimpleTransmission
-      </type>
+      <type>transmission_interface/SimpleTransmission</type>
+      <joint name="head_mount_head">
+        <hardwareInterface>EffortJointInterface</hardwareInterface>
+      </joint>
       <actuator name="head_mount_head_joint_actuator">
+        <hardwareInterface>EffortJointInterface</hardwareInterface>
         <mechanicalReduction>1</mechanicalReduction>
         <motorTorqueConstant>10</motorTorqueConstant>
-        <hardwareInterface>EffortJointInterface</hardwareInterface>
       </actuator>
       <!-- <mechanicalReduction>${-1 * 624/35 * 80/18}</mechanicalReduction> -->

File: ar600_description/urdf/head/head.urdf.xacro (robot description, xacro)
@@ -2,5 +2,5 @@
 <robot xmlns:xacro="http://ros.org/wiki/xacro">
 	<xacro:include filename="$(find ar600_description)/urdf/head/head.gazebo.xacro" />
-  	<!--<xacro:include filename="$(find ar600_description)/urdf/head/head.transmission.xacro" />-->
+  	<xacro:include filename="$(find ar600_description)/urdf/head/head.transmission.xacro" />
   	<xacro:macro name="ar600_head_xacro" params="name parent *origin">
   		<link name="${name}_link">
@@ -65,5 +65,5 @@
 			<origin xyz="0 0 0" rpy="0 0 0"/>
 		</joint>
-		<!--<xacro:ar600_head_transmission/>-->
+		<xacro:ar600_head_transmission/>
   	</xacro:macro>
 </robot>
